Commit message: successfully complete the visual and collision parameters of the whole robot. except inertia params

File: assets/robot_description/urdf/panda.xacro (robot description, xacro)
@@ -34,4 +34,5 @@
     <xacro:include filename="materials.xacro"/>
     <xacro:include filename="constants.xacro"/>
+    <!-- <link name="base"/> -->
     <xacro:panda parent="base" fx="0.28" fy="0.075" fz="0.005" bx="-0.03" by="0.04" bz="-0.05"/>
 </robot>

File: assets/robot_description/urdf/panda_arm/panda_arm_L6_LF.xacro (robot description, xacro)
@@ -1,5 +1,5 @@
 <?xml version="1.0"?>
 <robot xmlns:xacro="http://www.ros.org/wiki/xacro" name="panda">
-    <xacro:macro name="panda_arm_L6" params="prefix parent xyz rpy">
+    <xacro:macro name="panda_arm_L6_lf" params="prefix parent xyz rpy">
         <xacro:revolute_joint name="${prefix}_J6" parent="${parent}" child="${prefix}_L6" xyz="${xyz}" rpy="${rpy}" axis="1 0 0" />
         <link name="${prefix}_L6">
@@ -7,12 +7,13 @@
                 <origin xyz="0 0 0" rpy="0 0 0" />
                 <geometry>
-                    <mesh filename="${arm_mesh_path}/Link6.dae" scale="1 1 1" />
+                    <mesh filename="${arm_mesh_path}/Link6.dae" scale="-1 1 1" />
                 </geometry>
                 <material name="red" />
             </visual>
             <collision>
-                <origin xyz="0.0 0.0 -0.025" rpy="0 0 0" />
+                <origin xyz="0.0 0.0 0.0" rpy="0 0 0" />
                 <geometry>
-                    <cylinder radius="0.02" length="0.005"/>
+                    <!-- <cylinder radius="0.02" length="0.005"/> -->
+                    <mesh filename="${arm_mesh_path}/Link6.dae" scale="-1 1 1" />
                 </geometry>
             </collision>

File: assets/robot_description/urdf/panda_arm/panda_arm_L7.xacro (robot description, xacro)
@@ -2,17 +2,17 @@
 <robot xmlns:xacro="http://www.ros.org/wiki/xacro" name="panda">
     <xacro:macro name="panda_arm_L7" params="prefix parent xyz rpy">
-        <xacro:fixed_joint name="${prefix}_J7" parent="${parent}" child="${prefix}_L7" xyz="${xyz}" rpy="${rpy}"/>
+        <xacro:revolute_joint name="${prefix}_J7" parent="${parent}" child="${prefix}_L7" xyz="${xyz}" rpy="${rpy}" axis="1 0 0"/>
         <link name="${prefix}_L7">
             <visual>
                 <origin xyz="0 0 0" rpy="0 0 0" />
                 <geometry>
-                    <cylinder radius="0.01" length="0.005"/>
+                    <mesh filename="${arm_mesh_path}/Link7.dae" scale="1 1 1" />
                 </geometry>
-                <material name="blue" />
+                <!-- <material name="blue" /> -->
             </visual>
             <collision>
                 <origin xyz="0 0 0" rpy="0 0 0" />
                 <geometry>
-                    <cylinder radius="0.01" length="0.005"/>
+                    <mesh filename="${arm_mesh_path}/Link7.dae" scale="1 1 1" />
                 </geometry>
             </collision>

File: assets/robot_description/urdf/panda_arm/panda_arm_LF.xacro (robot description, xacro)
@@ -6,5 +6,5 @@
     <xacro:include filename="panda_arm_L4_LF.xacro"/>
     <xacro:include filename="panda_arm_L5.xacro"/>
-    <xacro:include filename="panda_arm_L6.xacro"/>
+    <xacro:include filename="panda_arm_L6_LF.xacro"/>
     <xacro:include filename="panda_arm_L7.xacro"/>
     <xacro:macro name="lf_arm" params="prefix parent xyz rpy">
@@ -15,6 +15,6 @@
         <xacro:panda_arm_L4_lf prefix="${prefix}" parent="${prefix}_L3" xyz="0.058 0.0195 0.001" rpy="0 ${pi/2} ${pi}"/>
         <xacro:panda_arm_L5 prefix="${prefix}" parent="${prefix}_L4" xyz="-0.0073 0.016 -0.04725" rpy="${pi/2} ${-pi/2} 0"/>
-        <xacro:panda_arm_L6 prefix="${prefix}" parent="${prefix}_L5" xyz="-0.065 0.021 0" rpy="0 ${pi/2} 0"/>
-        <xacro:panda_arm_L7 prefix="${prefix}" parent="${prefix}_L6" xyz="0 0 -0.031" rpy="0 0 0"/>
+        <xacro:panda_arm_L6_lf prefix="${prefix}" parent="${prefix}_L5" xyz="-0.065 0.021 0" rpy="0 ${pi/2} 0"/>
+        <xacro:panda_arm_L7 prefix="${prefix}" parent="${prefix}_L6" xyz="0 0.007 -0.08" rpy="0 0 0"/>
     </xacro:macro>
     <!--! TEST -->

File: assets/robot_description/urdf/panda_arm/panda_arm_RF.xacro (robot description, xacro)
@@ -6,5 +6,5 @@
     <xacro:include filename="panda_arm_L4_RF.xacro"/>
     <xacro:include filename="panda_arm_L5.xacro"/>
-    <xacro:include filename="panda_arm_L6.xacro"/>
+    <xacro:include filename="panda_arm_L6_RF.xacro"/>
     <xacro:include filename="panda_arm_L7.xacro"/>
     <xacro:macro name="rf_arm" params="prefix parent xyz rpy">
@@ -15,6 +15,6 @@
         <xacro:panda_arm_L4_rf prefix="${prefix}" parent="${prefix}_L3" xyz="0.058 0.0195 0.001" rpy="0 ${-pi/2} 0"/>
         <xacro:panda_arm_L5 prefix="${prefix}" parent="${prefix}_L4" xyz="-0.0073 -0.016 -0.04725" rpy="${pi/2} ${-pi/2} 0"/>
-        <xacro:panda_arm_L6 prefix="${prefix}" parent="${prefix}_L5" xyz="-0.065 0.021 0" rpy="0 ${pi/2} 0"/>
-        <xacro:panda_arm_L7 prefix="${prefix}" parent="${prefix}_L6" xyz="0 0 -0.031" rpy="0 0 0"/>
+        <xacro:panda_arm_L6_rf prefix="${prefix}" parent="${prefix}_L5" xyz="-0.065 0.021 0" rpy="0 ${pi/2} 0"/>
+        <xacro:panda_arm_L7 prefix="${prefix}" parent="${prefix}_L6" xyz="0 0.007 -0.08" rpy="0 0 0"/>
     </xacro:macro>
     <!--! TEST -->

File: assets/robot_description/urdf/panda_leg/panda_leg_L4_LB.xacro (robot description, xacro)
@@ -1,5 +1,5 @@
 <?xml version="1.0"?>
 <robot xmlns:xacro="http://www.ros.org/wiki/xacro" name="panda">
-    <xacro:macro name="panda_leg_L4" params="prefix parent xyz rpy">
+    <xacro:macro name="panda_leg_L4_lb" params="prefix parent xyz rpy">
         <xacro:revolute_joint name="${prefix}_J4" parent="${parent}" child="${prefix}_L4" xyz="${xyz}" rpy="${rpy}" axis="1 0 0" />
         <link name="${prefix}_L4">
@@ -7,12 +7,13 @@
                 <origin xyz="0 0 0" rpy="0 0 0" />
                 <geometry>
-                    <mesh filename="${leg_mesh_path}/Link4.dae" scale="1 1 1" />
+                    <mesh filename="${leg_mesh_path}/Link4.dae" scale="-1 1 1" />
                 </geometry>
                 <material name="red" />
             </visual>
              <collision>
-                <origin xyz="0.0 0.0 -0.025" rpy="0 0 0" />
+                <origin xyz="0.0 0.0 0.0" rpy="0 0 0" />
                 <geometry>
-                    <cylinder radius="0.02" length="0.005"/>
+                    <!-- <cylinder radius="0.02" length="0.005"/> -->
+                    <mesh filename="${leg_mesh_path}/Link4.dae" scale="-1 1 1" />
                 </geometry>
             </collision>

File: assets/robot_description/urdf/panda_leg/panda_leg_L5.xacro (robot description, xacro)
@@ -2,17 +2,17 @@
 <robot xmlns:xacro="http://www.ros.org/wiki/xacro" name="panda">
     <xacro:macro name="panda_leg_L5" params="prefix parent xyz rpy">
-        <xacro:fixed_joint name="${prefix}_J5" parent="${parent}" child="${prefix}_L5" xyz="${xyz}" rpy="${rpy}"/>
+        <xacro:revolute_joint name="${prefix}_J5" parent="${parent}" child="${prefix}_L5" xyz="${xyz}" rpy="${rpy}" axis="1 0 0"/>
         <link name="${prefix}_L5">
             <visual>
                 <origin xyz="0 0 0" rpy="0 0 0" />
                 <geometry>
-                    <cylinder radius="0.01" length="0.005"/>
+                    <mesh filename="${leg_mesh_path}/Link5.dae" scale="1 1 1" />
                 </geometry>
-                <material name="blue" />
+                <!-- <material name="blue" /> -->
             </visual>
             <collision>
                 <origin xyz="0 0 0" rpy="0 0 0" />
                 <geometry>
-                    <cylinder radius="0.01" length="0.005"/>
+                    <mesh filename="${leg_mesh_path}/Link5.dae" scale="1 1 1" />
                 </geometry>
             </collision>

File: assets/robot_description/urdf/panda_leg/panda_leg_LB.xacro (robot description, xacro)
@@ -4,5 +4,5 @@
     <xacro:include filename="panda_leg_L2_LB.xacro"/>
     <xacro:include filename="panda_leg_L3.xacro"/>
-    <xacro:include filename="panda_leg_L4.xacro"/>
+    <xacro:include filename="panda_leg_L4_LB.xacro"/>
     <xacro:include filename="panda_leg_L5.xacro"/>
     <xacro:macro name="lb_leg" params="prefix parent xyz rpy">
@@ -10,6 +10,6 @@
         <xacro:panda_leg_L2_lb prefix="${prefix}" parent="${prefix}_L1" xyz="-0.0485 0.00 -0.06210" rpy="0 -${pi/2} 0"/>
         <xacro:panda_leg_L3 prefix="${prefix}" parent="${prefix}_L2" xyz="-0.033 -0.11975 0.01875" rpy="${pi/2} ${pi} 0"/>
-        <xacro:panda_leg_L4 prefix="${prefix}" parent="${prefix}_L3" xyz="0.0 -0.09075 0.0" rpy="-${pi/2} 0 0"/>
-       <xacro:panda_leg_L5 prefix="${prefix}" parent="${prefix}_L4" xyz="0 0 -0.031" rpy="0 0 0"/>
+        <xacro:panda_leg_L4_lb prefix="${prefix}" parent="${prefix}_L3" xyz="0.0 -0.09075 0.0" rpy="-${pi/2} 0 0"/>
+       <xacro:panda_leg_L5 prefix="${prefix}" parent="${prefix}_L4" xyz="0 0.007 -0.08" rpy="0 0 0"/>
     </xacro:macro>
     <!--! TEST -->

File: assets/robot_description/urdf/panda_leg/panda_leg_RB.xacro (robot description, xacro)
@@ -4,5 +4,5 @@
     <xacro:include filename="panda_leg_L2_RB.xacro"/>
     <xacro:include filename="panda_leg_L3.xacro"/>
-    <xacro:include filename="panda_leg_L4.xacro"/>
+    <xacro:include filename="panda_leg_L4_RB.xacro"/>
     <xacro:include filename="panda_leg_L5.xacro"/>
     <xacro:macro name="rb_leg" params="prefix parent xyz rpy">
@@ -10,6 +10,6 @@
         <xacro:panda_leg_L2_rb prefix="${prefix}" parent="${prefix}_L1" xyz="-0.0485 0.00 -0.06210" rpy="${-pi} ${pi/2} 0"/>
         <xacro:panda_leg_L3 prefix="${prefix}" parent="${prefix}_L2" xyz="0.033 -0.11975 0.01875" rpy="${pi/2} ${pi} 0"/>
-        <xacro:panda_leg_L4 prefix="${prefix}" parent="${prefix}_L3" xyz="0.0 -0.09075 0.0" rpy="-${pi/2} 0 0"/>
-        <xacro:panda_leg_L5 prefix="${prefix}" parent="${prefix}_L4" xyz="0 0 -0.031" rpy="0 0 0"/>
+        <xacro:panda_leg_L4_rb prefix="${prefix}" parent="${prefix}_L3" xyz="0.0 -0.09075 0.0" rpy="-${pi/2} 0 0"/>
+        <xacro:panda_leg_L5 prefix="${prefix}" parent="${prefix}_L4" xyz="0 0.007 -0.08" rpy="0 0 0"/>
     </xacro:macro>
     <!--! TEST -->
