Commit message: feat: add inertia values to URDF and Gazebo visualization launch file
- Added inertia parameters to all arm, leg, and body xacro links
- Removed redundant panda_arm_L6.xacro from leg directory
- Added display_gazebo.launch.py for visualizing the robot in Gazebo

File: assets/robot_description/urdf/panda.urdf (robot description, URDF)
Before this commit: robot panda, 25 links, 24 joints
Links:
- link LB_L1: mass None -> 0.399; geometry collision cylinder length=0.075 radius=0.035; visual mesh filename=package://robot_description/meshes/panda_leg/Link1.dae scale=-1 1 1
- link LB_L2: mass None -> 0.29023; geometry collision cylinder length=0.16 radius=0.0275; visual mesh filename=package://robot_description/meshes/panda_leg/Link2.dae scale=1 1 -1
- link LB_L3: mass None -> 0.12; geometry collision cylinder length=0.055 radius=0.03; visual mesh filename=package://robot_description/meshes/panda_leg/Link3.dae scale=1 1 1
- link LB_L4: mass None -> 0.20986; geometry collision box size=0.065 0.02 0.06; visual mesh filename=package://robot_description/meshes/panda_leg/Link4.dae scale=-1 1 1
- link LB_L5: mass None -> 0.10248; geometry collision box size=0.08 0.02 0.05; visual mesh filename=package://robot_description/meshes/panda_leg/Link5.dae scale=1 1 1
- link LF_L1: mass None -> 0.21205; geometry collision cylinder length=0.085 radius=0.025; visual mesh filename=package://robot_description/meshes/panda_arm/Link1.dae scale=1 1 1
- link LF_L2: mass None -> 0.12339; geometry collision cylinder length=0.04 radius=0.025; visual mesh filename=package://robot_description/meshes/panda_arm/Link2.dae scale=1 1 1
- link LF_L3: mass None -> 0.02605; geometry collision cylinder length=0.01 radius=0.025; visual mesh filename=package://robot_description/meshes/panda_arm/Link3.dae scale=1 1 1
- link LF_L4: mass None -> 0.21197; geometry collision cylinder length=0.05 radius=0.03; visual mesh filename=package://robot_description/meshes/panda_arm/Link4.dae scale=1 -1 1
- link LF_L5: mass None -> 0.11428; geometry collision cylinder length=0.0525 radius=0.0175; visual mesh filename=package://robot_description/meshes/panda_arm/Link5.dae scale=1 1 1
- link LF_L6: mass None -> 0.20986; geometry collision box size=0.065 0.02 0.06; visual mesh filename=package://robot_description/meshes/panda_arm/Link6.dae scale=-1 1 1
- link LF_L7: mass None -> 0.10248; geometry collision box size=0.08 0.02 0.05; visual mesh filename=package://robot_description/meshes/panda_arm/Link7.dae scale=1 1 1
- link RB_L1: mass None -> 0.399; geometry collision cylinder length=0.075 radius=0.035; visual mesh filename=package://robot_description/meshes/panda_leg/Link1.dae scale=-1 1 1
- link RB_L2: mass None -> 0.29023; geometry collision cylinder length=0.16 radius=0.0275; visual mesh filename=package://robot_description/meshes/panda_leg/Link2.dae scale=-1 1 -1
- link RB_L3: mass None -> 0.12; geometry collision cylinder length=0.055 radius=0.03; visual mesh filename=package://robot_description/meshes/panda_leg/Link3.dae scale=1 1 1
- link RB_L4: mass None -> 0.20986; geometry collision box size=0.065 0.02 0.06; visual mesh filename=package://robot_description/meshes/panda_leg/Link4.dae scale=1 1 1
- link RB_L5: mass None -> 0.10248; geometry collision box size=0.08 0.02 0.05; visual mesh filename=package://robot_description/meshes/panda_leg/Link5.dae scale=1 1 1
- link RF_L1: mass None -> 0.21205; geometry collision cylinder length=0.085 radius=0.025; visual mesh filename=package://robot_description/meshes/panda_arm/Link1.dae scale=1 1 1
- link RF_L2: mass None -> 0.12339; geometry collision cylinder length=0.04 radius=0.025; visual mesh filename=package://robot_description/meshes/panda_arm/Link2.dae scale=1 1 1
- link RF_L3: mass None -> 0.02605; geometry collision cylinder length=0.01 radius=0.025; visual mesh filename=package://robot_description/meshes/panda_arm/Link3.dae scale=1 1 1
- link RF_L4: mass None -> 0.21197; geometry collision cylinder length=0.05 radius=0.03; visual mesh filename=package://robot_description/meshes/panda_arm/Link4.dae scale=1 1 1
- link RF_L5: mass None -> 0.11428; geometry collision cylinder length=0.0525 radius=0.0175; visual mesh filename=package://robot_description/meshes/panda_arm/Link5.dae scale=1 1 1
- link RF_L6: mass None -> 0.20986; geometry collision box size=0.065 0.02 0.06; visual mesh filename=package://robot_description/meshes/panda_arm/Link6.dae scale=1 1 1
- link RF_L7: mass None -> 0.10248; geometry collision box size=0.08 0.02 0.05; visual mesh filename=package://robot_description/meshes/panda_arm/Link7.dae scale=1 1 1
- link body: mass None -> 0.6; geometry collision cylinder length=0.04 radius=0.06; collision cylinder length=0.125 radius=0.045
Joints:
- joint LB_J1: origin xyz=-0.02500000000000001 -0.2 0 rpy=1.5707963267948966 0 1.5707963267948966 -> xyz=-0.03 0.04 -0.05 rpy=1.5707963267948966 0 0
- joint LB_J3: origin xyz=-0.033 -0.11975 -0.01875 rpy=-1.5707963267948966 3.141592653589793 0 -> xyz=-0.033 -0.11975 0.01875 rpy=1.5707963267948966 3.141592653589793 0
- joint LB_J5: axis (none) -> 1 0 0; limit (none) -> lower=-1.5707963267948966 upper=1.5707963267948966 effort=10.0 velocity=10.0; origin xyz=0 0 -0.031 rpy=0 0 0 -> xyz=0 0.007 -0.08 rpy=0 0 0; type fixed -> revolute
- joint LF_J1: origin xyz=-0.1 0.15 0 rpy=0 0 3.141592653589793 -> xyz=0.28 0.075 0.005 rpy=0 0 1.5707963267948966
- joint LF_J4: origin xyz=0.058 0.0195 0.001 rpy=-1.5707963267948966 1.5707963267948966 3.141592653589793 -> xyz=0.058 0.0195 0.001 rpy=0 1.5707963267948966 3.141592653589793
- joint LF_J7: axis (none) -> 1 0 0; limit (none) -> lower=-1.5707963267948966 upper=1.5707963267948966 effort=10.0 velocity=10.0; origin xyz=0 0 -0.031 rpy=0 0 0 -> xyz=0 0.007 -0.08 rpy=0 0 0; type fixed -> revolute
- joint RB_J1: origin xyz=0.02500000000000001 -0.2 0 rpy=-1.5707963267948966 0 1.5707963267948966 -> xyz=-0.03 -0.04 -0.05 rpy=-1.5707963267948966 0 0
- joint RB_J3: origin xyz=0.033 -0.11975 -0.01875 rpy=-1.5707963267948966 3.141592653589793 0 -> xyz=0.033 -0.11975 0.01875 rpy=1.5707963267948966 3.141592653589793 0
- joint RB_J5: axis (none) -> 1 0 0; limit (none) -> lower=-1.5707963267948966 upper=1.5707963267948966 effort=10.0 velocity=10.0; origin xyz=0 0 -0.031 rpy=0 0 0 -> xyz=0 0.007 -0.08 rpy=0 0 0; type fixed -> revolute
- joint RF_J1: origin xyz=0.1 0.15 0 rpy=0 0 0 -> xyz=0.28 -0.075 0.005 rpy=0 0 -1.5707963267948966
- joint RF_J4: origin xyz=0.058 0.0195 0.001 rpy=1.5707963267948966 -1.5707963267948966 0 -> xyz=0.058 0.0195 0.001 rpy=0 -1.5707963267948966 0
- joint RF_J7: axis (none) -> 1 0 0; limit (none) -> lower=-1.5707963267948966 upper=1.5707963267948966 effort=10.0 velocity=10.0; origin xyz=0 0 -0.031 rpy=0 0 0 -> xyz=0 0.007 -0.08 rpy=0 0 0; type fixed -> revolute

File: assets/robot_description/urdf/panda_arm/panda_arm_L1.xacro (robot description, xacro)
@@ -17,4 +17,12 @@
                 </geometry>
             </collision>
+            <inertial>
+                <origin xyz="0.024340 0.000290 -0.009336" rpy="0 0 0"/>
+                <mass value="0.21205"/>
+                <inertia
+                    ixx="0.00014885" ixy="-0.00000038" ixz="0.00000863"
+                    iyy="0.00012057" iyz="0.00000411"
+                    izz="0.00009025"/>
+            </inertial>
         </link>
     </xacro:macro>

File: assets/robot_description/urdf/panda_arm/panda_arm_L2.xacro (robot description, xacro)
@@ -17,4 +17,12 @@
                 </geometry>
             </collision>
+            <inertial>
+                <origin xyz="0.000319 0.007895 -0.042269" rpy="0 0 0"/>
+                <mass value="0.12339"/>
+                <inertia
+                    ixx="0.00007467" ixy="0.00000015" ixz="-0.00000018"
+                    iyy="0.00007863" iyz="0.00000833"
+                    izz="0.00005700"/>
+            </inertial>
         </link>
     </xacro:macro>

File: assets/robot_description/urdf/panda_arm/panda_arm_L3.xacro (robot description, xacro)
@@ -17,4 +17,12 @@
                 </geometry>
             </collision>
+            <inertial>
+                <origin xyz="0.017019 0.023760 -0.000188" rpy="0 0 0"/>
+                <mass value="0.02605"/>
+                <inertia
+                    ixx="0.00000523" ixy="0.00000090" ixz="0.00000009"
+                    iyy="0.00013027" iyz="0.00000007"
+                    izz="0.00001104"/>
+            </inertial>
         </link>
     </xacro:macro>

File: assets/robot_description/urdf/panda_arm/panda_arm_L4_LF.xacro (robot description, xacro)
@@ -17,4 +17,12 @@
                 </geometry>
             </collision>
+            <inertial>
+                <origin xyz="0.005528 0.015452 -0.024028" rpy="0 0 0"/>
+                <mass value="0.21197"/>
+                <inertia
+                    ixx="0.00016760" ixy="0.00000028" ixz="0.00001932"
+                    iyy="0.00017551" iyz="0.00000051"
+                    izz="0.00008108"/>
+            </inertial>
         </link>
     </xacro:macro>

File: assets/robot_description/urdf/panda_arm/panda_arm_L4_RF.xacro (robot description, xacro)
@@ -17,4 +17,12 @@
                 </geometry>
             </collision>
+            <inertial>
+                <origin xyz="0.005528 -0.015452 -0.024028" rpy="0 0 0"/>
+                <mass value="0.21197"/>
+                <inertia
+                    ixx="0.00016760" ixy="-0.00000028" ixz="0.00001932"
+                    iyy="0.00017551" iyz="-0.00000051"
+                    izz="0.00008108"/>
+            </inertial>
         </link>
     </xacro:macro>

File: assets/robot_description/urdf/panda_arm/panda_arm_L5.xacro (robot description, xacro)
@@ -17,4 +17,12 @@
                 </geometry>
             </collision>
+            <inertial>
+                <origin xyz="-0.039812 0.022259 -0.000292" rpy="0 0 0"/>
+                <mass value="0.11428"/>
+                <inertia
+                    ixx="0.00002245" ixy="-0.00000489" ixz="-0.00000014"
+                    iyy="0.00008311" iyz="-0.00000020"
+                    izz="0.00007996"/>
+            </inertial>
         </link>
     </xacro:macro>

File: assets/robot_description/urdf/panda_arm/panda_arm_L6_LF.xacro (robot description, xacro)
@@ -17,4 +17,12 @@
                 </geometry>
             </collision>
+            <inertial>
+                <origin xyz="0.005400 0.000762 -0.054807" rpy="0 0 0"/>
+                <mass value="0.20986"/>
+                <inertia
+                    ixx="0.00011473" ixy="0.00001510" ixz="-0.00000999"
+                    iyy="0.00017398" iyz="0.00001411"
+                    izz="0.00013573"/>
+            </inertial>
         </link>
     </xacro:macro>

File: assets/robot_description/urdf/panda_arm/panda_arm_L6_RF.xacro (robot description, xacro)
@@ -17,4 +17,12 @@
                 </geometry>
             </collision>
+            <inertial>
+                <origin xyz="-0.005400 0.000762 -0.054807" rpy="0 0 0"/>
+                <mass value="0.20986"/>
+                <inertia
+                    ixx="0.00011473" ixy="-0.00001510" ixz="0.00000999"
+                    iyy="0.00017398" iyz="0.00001411"
+                    izz="0.00013573" />
+            </inertial>
         </link>
     </xacro:macro>

File: assets/robot_description/urdf/panda_arm/panda_arm_L7.xacro (robot description, xacro)
@@ -23,4 +23,12 @@
                 </geometry>
             </collision>
+            <inertial>
+                <origin xyz="0.001048 -0.007730 -0.047829" rpy="0 0 0"/>
+                <mass value="0.10248"/>
+                <inertia
+                    ixx="0.00003528" ixy="-0.00000068" ixz="-0.00000123"
+                    iyy="0.00007729" iyz="-0.00000298"
+                    izz="0.00005640"/>
+            </inertial>
         </link>
     </xacro:macro>

File: assets/robot_description/urdf/panda_body/panda_body.xacro (robot description, xacro)
@@ -28,4 +28,12 @@
                 </geometry>
             </collision>
+            <inertial>
+                <origin xyz="0.111021 0.001066 -0.054499" rpy="0 0 0"/>
+                <mass value="0.6"/>
+                <inertia
+                    ixx="0.00341830" ixy="-0.00001942" ixz="-0.00061387"
+                    iyy="0.00715863" iyz="-0.00000747"
+                    izz="0.00795982"/>
+            </inertial>
         </link>
     </xacro:macro>

File: assets/robot_description/urdf/panda_leg/panda_leg_L1.xacro (robot description, xacro)
@@ -17,4 +17,13 @@
                 </geometry>
             </collision>
+            <!-- X-flipped mesh (scale="-1 1 1"): CoM x negated, ixy and ixz negated -->
+            <inertial>
+                <origin xyz="-0.028971 -0.000107 -0.018559" rpy="0 0 0"/>
+                <mass value="0.399"/>
+                <inertia
+                    ixx="0.00032351" ixy="-0.00000101" ixz="-0.00001007"
+                    iyy="0.00030113" iyz="-0.00000164"
+                    izz="0.00031142"/>
+            </inertial>
         </link>
     </xacro:macro>

File: assets/robot_description/urdf/panda_leg/panda_leg_L2_LB.xacro (robot description, xacro)
@@ -17,4 +17,12 @@
                 </geometry>
             </collision>
+            <inertial>
+                <origin xyz="-0.028482 -0.066047 0.001028" rpy="0 0 0"/>
+                <mass value="0.29023"/>
+                <inertia
+                    ixx="0.00085932" ixy="-0.00007468" ixz="-0.00000037"
+                    iyy="0.00016110" iyz="-0.00000441"
+                    izz="0.00081281"/>
+            </inertial>
         </link>
     </xacro:macro>

File: assets/robot_description/urdf/panda_leg/panda_leg_L2_RB.xacro (robot description, xacro)
@@ -17,4 +17,12 @@
                 </geometry>
             </collision>
+            <inertial>
+                <origin xyz="0.028482 -0.066047 0.001028" rpy="0 0 0"/>
+                <mass value="0.29023"/>
+                <inertia
+                    ixx="0.00085932" ixy="0.00007468" ixz="0.00000037"
+                    iyy="0.00016110" iyz="-0.00000441"
+                    izz="0.00081281"/>
+            </inertial>
         </link>
     </xacro:macro>

File: assets/robot_description/urdf/panda_leg/panda_leg_L3.xacro (robot description, xacro)
@@ -17,4 +17,12 @@
                 </geometry>
             </collision>
+            <inertial>
+                <origin xyz="0.000069 -0.055725 0.001186" rpy="0 0 0"/>
+                <mass value="0.12"/>
+                <inertia
+                    ixx="0.00009751" ixy="0.00000010" ixz="-0.00000012"
+                    iyy="0.00005226" iyz="0.00000224"
+                    izz="0.00012515"/>
+            </inertial>
         </link>
     </xacro:macro>

File: assets/robot_description/urdf/panda_leg/panda_leg_L4_LB.xacro (robot description, xacro)
@@ -17,4 +17,12 @@
                 </geometry>
             </collision>
+            <inertial>
+                <origin xyz="0.005400 0.000762 -0.054807" rpy="0 0 0"/>
+                <mass value="0.20986"/>
+                <inertia
+                    ixx="0.00011473" ixy="0.00001510" ixz="-0.00000999"
+                    iyy="0.00017398" iyz="0.00001411"
+                    izz="0.00013573"/>
+            </inertial>
         </link>
     </xacro:macro>

File: assets/robot_description/urdf/panda_leg/panda_leg_L4_RB.xacro (robot description, xacro)
@@ -17,4 +17,12 @@
                 </geometry>
             </collision>
+            <inertial>
+                <origin xyz="-0.005400 0.000762 -0.054807" rpy="0 0 0"/>
+                <mass value="0.20986"/>
+                <inertia
+                    ixx="0.00011473" ixy="-0.00001510" ixz="0.00000999"
+                    iyy="0.00017398" iyz="0.00001411"
+                    izz="0.00013573" />
+            </inertial>
         </link>
     </xacro:macro>

File: assets/robot_description/urdf/panda_leg/panda_leg_L5.xacro (robot description, xacro)
@@ -19,4 +19,12 @@
                 </geometry>
             </collision>
+            <inertial>
+                <origin xyz="0.001048 -0.007730 -0.047829" rpy="0 0 0"/>
+                <mass value="0.10248"/>
+                <inertia
+                    ixx="0.00003528" ixy="-0.00000068" ixz="-0.00000123"
+                    iyy="0.00007729" iyz="-0.00000298"
+                    izz="0.00005640"/>
+            </inertial>
         </link>
     </xacro:macro>
