Commit message: refactor: simplify panda palm's collision matrix, use simple geometry to simplify the system calculation.

File: assets/robot_description/urdf/panda_arm/panda_arm_L6_LF.xacro (robot description, xacro)
@@ -12,8 +12,7 @@
             </visual>
             <collision>
-                <origin xyz="0.0 0.0 0.0" rpy="0 0 0" />
+                <origin xyz="0.0 0.0 -0.06" rpy="0 0 0" />
                 <geometry>
-                    <!-- <cylinder radius="0.02" length="0.005"/> -->
-                    <mesh filename="${arm_mesh_path}/Link6.dae" scale="-1 1 1" />
+                    <box size="0.065 0.02 0.06"/> <!-- TODO: set x y z size -->
                 </geometry>
             </collision>

File: assets/robot_description/urdf/panda_arm/panda_arm_L6_RF.xacro (robot description, xacro)
@@ -12,8 +12,7 @@
             </visual>
             <collision>
-                <origin xyz="0.0 0.0 0.0" rpy="0 0 0" />
+                <origin xyz="0.0 0.0 -0.06" rpy="0 0 0" />
                 <geometry>
-                    <!-- <cylinder radius="0.02" length="0.005"/> -->
-                    <mesh filename="${arm_mesh_path}/Link6.dae" scale="1 1 1" />
+                    <box size="0.065 0.02 0.06"/> <!-- TODO: set x y z size -->
                 </geometry>
             </collision>

File: assets/robot_description/urdf/panda_arm/panda_arm_L7.xacro (robot description, xacro)
@@ -12,7 +12,13 @@
             </visual>
             <collision>
-                <origin xyz="0 0 0" rpy="0 0 0" />
+                <!-- <origin xyz="0 0 0" rpy="0 0 0" />
                 <geometry>
                     <mesh filename="${arm_mesh_path}/Link7.dae" scale="1 1 1" />
+                </geometry> -->
+                <origin xyz="0.0 0.0 -0.05" rpy="0 0 0" />
+                <geometry>
+                    <!-- <mesh filename="${meshes_path}/Link5.dae" scale="${reflect} 1 1" /> -->
+                    <!-- <cylinder radius="0.015" length="0.07"/> -->
+                    <box size="0.08 0.02 0.05"/> <!-- TODO: set x y z size -->
                 </geometry>
             </collision>

File: assets/robot_description/urdf/panda_leg/panda_leg_L4_LB.xacro (robot description, xacro)
@@ -12,8 +12,7 @@
             </visual>
              <collision>
-                <origin xyz="0.0 0.0 0.0" rpy="0 0 0" />
+                <origin xyz="0.0 0.0 -0.06" rpy="0 0 0" />
                 <geometry>
-                    <!-- <cylinder radius="0.02" length="0.005"/> -->
-                    <mesh filename="${leg_mesh_path}/Link4.dae" scale="-1 1 1" />
+                    <box size="0.065 0.02 0.06"/> <!-- TODO: set x y z size -->
                 </geometry>
             </collision>

File: assets/robot_description/urdf/panda_leg/panda_leg_L4_RB.xacro (robot description, xacro)
@@ -12,8 +12,7 @@
             </visual>
              <collision>
-                <origin xyz="0.0 0.0 0.0" rpy="0 0 0" />
+                <origin xyz="0.0 0.0 -0.06" rpy="0 0 0" />
                 <geometry>
-                    <!-- <cylinder radius="0.02" length="0.005"/> -->
-                    <mesh filename="${leg_mesh_path}/Link4.dae" scale="1 1 1" />
+                    <box size="0.065 0.02 0.06"/> <!-- TODO: set x y z size -->
                 </geometry>
             </collision>

File: assets/robot_description/urdf/panda_leg/panda_leg_L5.xacro (robot description, xacro)
@@ -12,7 +12,9 @@
             </visual>
             <collision>
-                <origin xyz="0 0 0" rpy="0 0 0" />
+                <origin xyz="0.0 0.0 -0.05" rpy="0 0 0" />
                 <geometry>
-                    <mesh filename="${leg_mesh_path}/Link5.dae" scale="1 1 1" />
+                    <!-- <mesh filename="${meshes_path}/Link5.dae" scale="${reflect} 1 1" /> -->
+                    <!-- <cylinder radius="0.015" length="0.07"/> -->
+                    <box size="0.08 0.02 0.05"/> <!-- TODO: set x y z size -->
                 </geometry>
             </collision>
